Commit message: adds node for simulator, fixes camera position in urdf

File: urdf/quadrotor_with_upward_facing_cam.urdf.xacro (robot description, xacro)
@@ -12,5 +12,5 @@
     <xacro:include filename="$(find hector_sensors_description)/urdf/generic_camera.urdf.xacro" />
     <xacro:generic_camera name="downward_cam" parent="base_link" ros_topic="camera/image" cam_info_topic="camera/camera_info" update_rate="20" res_x="640" res_y="480" image_format="L8" hfov="100">
-      <origin xyz="0.4 0.0 1.0" rpy="0 ${-M_PI/2} 0"/>
+      <origin xyz="0.0 0.0 1.0" rpy="0 ${-M_PI/2} 0"/>
     </xacro:generic_camera>
 </robot>
